Commit message: Refactor launch files and scripts for YOLOv5 integration
- Refactor the launch file `sunday_bringup_moveit.launch` to remove unnecessary whitespace and commented out code.
- Update the launch file `yolo_v5.launch` in the `yolov5_ros` package to set the `use_cpu` parameter to `true`.
- Modify the `sunday_trajectory_control.yaml` file to update the gains for the arm joints.
- Update the `grasp.py` script in the `sunday_gazebo` package to fix a bug in the `compute_cartesian_path` function.

File: src/sunday/sunday_description/urdf/sunday.xacro (robot description, xacro)
@@ -1,9 +1,10 @@
 <?xml version="1.0" encoding="utf-8"?>
-<!-- This URDF was automatically created by SolidWorks to URDF Exporter! Originally created by Stephen Brawner (brawner@gmail.com)
+<!-- This URDF was automatically created by SolidWorks to URDF Exporter! Originally created by
+Stephen Brawner (brawner@gmail.com)
      Commit Version: 1.5.1-0-g916b5db  Build Version: 1.5.7152.31018
      For more information, please see http://wiki.ros.org/sw_urdf_exporter -->
 <robot name="sunday" xmlns:xacro="http://ros.org/wiki/xacro">
-    <link name="base_footprint">
-    </link>
+  <link name="base_footprint">
+  </link>
   <link name="base_link">
     <inertial>
@@ -11,6 +12,6 @@
         xyz="-0.0041595 -0.019776 0.12"
         rpy="0 0 0" />
-        <mass value="0.524001417146026" />
-        <inertia ixx="1" ixy="0" ixz="0" iyy="1" iyz="0" izz="1" />
+      <mass value="0.524001417146026" />
+      <inertia ixx="1" ixy="0" ixz="0" iyy="1" iyz="0" izz="1" />
     </inertial>
     <visual>
@@ -38,9 +39,9 @@
     </collision>
   </link>
-    <joint name="base_link2base_footprint" type="fixed">
-        <parent link="base_footprint" />
-        <child link="base_link"/>
-        <origin xyz="0 0 0.032" rpy="0 0 0" />
-    </joint>
+  <joint name="base_link2base_footprint" type="fixed">
+    <parent link="base_footprint" />
+    <child link="base_link" />
+    <origin xyz="0 0 0.032" rpy="0 0 0" />
+  </joint>
   <link name="link_1">
     <inertial>
@@ -48,6 +49,6 @@
         xyz="4.4076E-07 0.0088489 0.03981"
         rpy="0 0 0" />
-        <mass value="0.166259789544396" />
-        <inertia ixx="1" ixy="0" ixz="0" iyy="1" iyz="0" izz="1" />
+      <mass value="0.166259789544396" />
+      <inertia ixx="1" ixy="0" ixz="0" iyy="1" iyz="0" izz="1" />
     </inertial>
     <visual>
@@ -99,6 +100,6 @@
         xyz="5.2117E-07 0.050183 0.046384"
         rpy="0 0 0" />
-        <mass value="0.316094041078938" />
-        <inertia ixx="1" ixy="0" ixz="0" iyy="1" iyz="0" izz="1" />
+      <mass value="0.316094041078938" />
+      <inertia ixx="1" ixy="0" ixz="0" iyy="1" iyz="0" izz="1" />
     </inertial>
     <visual>
@@ -150,6 +151,6 @@
         xyz="-2.3744E-06 0.013658 -0.095655"
         rpy="0 0 0" />
-        <mass value="0.323135746651779" />
-        <inertia ixx="1" ixy="0" ixz="0" iyy="1" iyz="0" izz="1" />
+      <mass value="0.323135746651779" />
+      <inertia ixx="1" ixy="0" ixz="0" iyy="1" iyz="0" izz="1" />
     </inertial>
     <visual>
@@ -201,6 +202,6 @@
         xyz="-6.4344E-06 -0.026419 -0.014391"
         rpy="0 0 0" />
-        <mass value="0.174947986817189" />
-        <inertia ixx="1" ixy="0" ixz="0" iyy="1" iyz="0" izz="1" />
+      <mass value="0.174947986817189" />
+      <inertia ixx="1" ixy="0" ixz="0" iyy="1" iyz="0" izz="1" />
     </inertial>
     <visual>
@@ -252,6 +253,6 @@
         xyz="0.00020466 -0.017155 -0.036587"
         rpy="0 0 0" />
-        <mass value="0.174947985033356" />
-        <inertia ixx="1" ixy="0" ixz="0" iyy="1" iyz="0" izz="1" />
+      <mass value="0.174947985033356" />
+      <inertia ixx="1" ixy="0" ixz="0" iyy="1" iyz="0" izz="1" />
     </inertial>
     <visual>
@@ -401,37 +402,37 @@
       xyz="0 0 0" />
   </joint> -->
-<!-- Used for fixing robot to Gazebo 'base_link' -->
-  <link name="world"/>
+  <!-- Used for fixing robot to Gazebo 'base_link' -->
+  <link name="world" />
   <joint name="fixed" type="fixed">
     <origin
       xyz="0 0 1.1"
       rpy="0 0 0" />
-    <parent link="world"/>
-    <child link="base_footprint"/>
+    <parent link="world" />
+    <child link="base_footprint" />
   </joint>
   <!-- <xacro:include filename="$(find sunday_description)/urdf/realsense/realsense.xacro"/> -->
-<xacro:include filename="$(find realsense_ros_gazebo)/xacro/depthcam.xacro"/>
-<xacro:realsense_d435 sensor_name="camera" parent_link="link_5" rate="30">
-    <origin xyz="-0.00068847 -0.06 -0.13" rpy="-3.14 0 -1.5708"/>
-</xacro:realsense_d435>
-<!-- Transmissions for ROS Control -->
-<xacro:macro name="transmission_block" params="joint_name">
-  <transmission name="tran1">
-    <type>transmission_interface/SimpleTransmission</type>
-    <joint name="${joint_name}">
-      <hardwareInterface>hardware_interface/PositionJointInterface</hardwareInterface>
-    </joint>
-    <actuator name="motor1">
-      <hardwareInterface>hardware_interface/PositionJointInterface</hardwareInterface>
-      <mechanicalReduction>1</mechanicalReduction>
-    </actuator>
-  </transmission>
-</xacro:macro>
-<xacro:transmission_block joint_name="joint_1"/>
-<xacro:transmission_block joint_name="joint_2"/>
-<xacro:transmission_block joint_name="joint_3"/>
-<xacro:transmission_block joint_name="joint_4"/>
-<xacro:transmission_block joint_name="joint_5"/>
-<xacro:transmission_block joint_name="joint_6"/>
+  <xacro:include filename="$(find realsense_ros_gazebo)/xacro/depthcam.xacro" />
+  <xacro:realsense_d435 sensor_name="camera" parent_link="link_5" rate="30">
+    <origin xyz="-0.00068847 -0.06 -0.13" rpy="-3.14 0 -1.5708" />
+  </xacro:realsense_d435>
+  <!-- Transmissions for ROS Control -->
+  <xacro:macro name="transmission_block" params="joint_name">
+    <transmission name="tran1">
+      <type>transmission_interface/SimpleTransmission</type>
+      <joint name="${joint_name}">
+        <hardwareInterface>hardware_interface/PositionJointInterface</hardwareInterface>
+      </joint>
+      <actuator name="motor1">
+        <hardwareInterface>hardware_interface/PositionJointInterface</hardwareInterface>
+        <mechanicalReduction>1</mechanicalReduction>
+      </actuator>
+    </transmission>
+  </xacro:macro>
+  <xacro:transmission_block joint_name="joint_1" />
+  <xacro:transmission_block joint_name="joint_2" />
+  <xacro:transmission_block joint_name="joint_3" />
+  <xacro:transmission_block joint_name="joint_4" />
+  <xacro:transmission_block joint_name="joint_5" />
+  <xacro:transmission_block joint_name="joint_6" />
   <!-- ros_control plugin -->
   <gazebo>
@@ -444,5 +445,6 @@
   <!-- vacuum_gripper plugin -->
   <gazebo>
-    <plugin name="gazebo_ros_vacuum_gripper" filename="libvacuum_plugin.so">
+    <plugin name="gazebo_ros_vacuum_gripper_debugger"
+      filename="libgazebo_ros_vacuum_gripper_debugger.so">
       <robotNamespace>/sunday/vacuum_gripper</robotNamespace>
       <bodyName>link_6</bodyName>
@@ -451,13 +453,13 @@
       <minDistance>0.03</minDistance>
     </plugin>
-</gazebo>
-<gazebo reference="link_6">
-  <mu1>50</mu1>
-  <mu2>50</mu2>
-  <minDepth>0.003</minDepth>
-  <maxVel>0</maxVel>
-  <kp>1000000.0</kp>
-  <kd>1.0</kd>
-  <material>Gazebo/Grey</material>
-</gazebo>
+  </gazebo>
+  <gazebo reference="link_6">
+    <mu1>50</mu1>
+    <mu2>50</mu2>
+    <minDepth>0.003</minDepth>
+    <maxVel>0</maxVel>
+    <kp>1000000.0</kp>
+    <kd>1.0</kd>
+    <material>Gazebo/Grey</material>
+  </gazebo>
 </robot>
