Commit message: Refactor launch files for YOLOv5 integration and robot navigation

File: src/my_robot_navigation/urdf/xacro/base_wheel.xacro (robot description, xacro)
@@ -123,3 +123,11 @@
     <xacro:add_support_wheel name="front" flag="1" />
     <xacro:add_support_wheel name="back" flag="-1" />
+    <!-- 包含sunday机械臂 -->
+    <xacro:include filename="path/to/sunday.xacro" />
+    <!-- 设置base_link和sunday之间的连接 -->
+    <joint name="base_to_sunday" type="fixed">
+        <parent link="base_link" /> <!-- base_wheel的基链接 -->
+        <child link="base_footprint" /> <!-- sunday的基链接 -->
+        <origin xyz="0 0 ${base_link_length / 2}" rpy="0 0 0" /> <!-- 根据需要调整位置和姿态 -->
+    </joint>
 </robot>

File: src/my_robot_navigation/urdf/xacro/camera.xacro (robot description, xacro)
@@ -42,5 +42,5 @@
         <material>Gazebo/Blue</material>
     </gazebo>
-    <!-- <gazebo reference="kinect link名称"> -->
+    <!-- <gazebo reference="kinectic link名称"> -->
     <gazebo reference="camera">
         <sensor type="depth" name="camera">

Commit message: Refactor launch files and scripts for YOLOv5 integration

File: src/my_robot_navigation/urdf/xacro/base_wheel.xacro (robot description, xacro)
@@ -9,21 +9,21 @@
     </material>
     <!-- 底盘属性 -->
-    <xacro:property name="base_footprint_radius" value="0.001" /> <!-- base_footprint 半径  -->
-    <xacro:property name="base_link_radius" value="0.1" /> <!-- base_link 半径 -->
-    <xacro:property name="base_link_length" value="0.08" /> <!-- base_link 长 -->
+    <xacro:property name="base_wheel_footprint_radius" value="0.001" /> <!-- base_wheel_footprint 半径  -->
+    <xacro:property name="base_wheel_link_radius" value="0.1" /> <!-- base_wheel_link 半径 -->
+    <xacro:property name="base_wheel_link_length" value="0.08" /> <!-- base_wheel_link 长 -->
     <xacro:property name="earth_space" value="0.015" /> <!-- 离地间距 -->
-    <xacro:property name="base_link_m" value="0.5" /> <!-- 质量  -->
+    <xacro:property name="base_wheel_link_m" value="0.5" /> <!-- 质量  -->
     <!-- 底盘 -->
-    <link name="base_footprint">
+    <link name="base_wheel_footprint">
         <visual>
             <geometry>
-                <sphere radius="${base_footprint_radius}" />
+                <sphere radius="${base_wheel_footprint_radius}" />
             </geometry>
         </visual>
     </link>
-    <link name="base_link">
+    <link name="base_wheel_link">
         <visual>
             <geometry>
-                <cylinder radius="${base_link_radius}" length="${base_link_length}" />
+                <cylinder radius="${base_wheel_link_radius}" length="${base_wheel_link_length}" />
             </geometry>
             <origin xyz="0 0 0" rpy="0 0 0" />
@@ -35,18 +35,18 @@
         <collision>
             <geometry>
-                <cylinder radius="${base_link_radius}" length="${base_link_length}" />
+                <cylinder radius="${base_wheel_link_radius}" length="${base_wheel_link_length}" />
             </geometry>
             <origin xyz="0 0 0" rpy="0 0 0" />
         </collision>
         <!-- 与rviz不同（2）：使用在head.xacro中封装过的inertial标签 -->
-        <xacro:cylinder_inertial_matrix m="${base_link_m}" r="${base_link_radius}"
-            h="${base_link_length}" />
+        <xacro:cylinder_inertial_matrix m="${base_wheel_link_m}" r="${base_wheel_link_radius}"
+            h="${base_wheel_link_length}" />
     </link>
-    <joint name="base_link2base_footprint" type="fixed">
-        <parent link="base_footprint" />
-        <child link="base_link" />
-        <origin xyz="0 0 ${earth_space + base_link_length / 2 }" />
+    <joint name="base_wheel_link2base_wheel_footprint" type="fixed">
+        <parent link="base_wheel_footprint" />
+        <child link="base_wheel_link" />
+        <origin xyz="0 0 ${earth_space + base_wheel_link_length / 2 }" />
     </joint>
-    <gazebo reference="base_link">
+    <gazebo reference="base_wheel_link">
         <!-- 与rviz不同（3）：重新设置颜色 -->
         <material>Gazebo/Yellow</material>
@@ -75,9 +75,9 @@
             <xacro:cylinder_inertial_matrix m="${wheel_m}" r="${wheel_radius}" h="${wheel_length}" />
         </link>
-        <joint name="${name}_wheel2base_link" type="continuous">
-            <parent link="base_link" />
+        <joint name="${name}_wheel2base_wheel_link" type="continuous">
+            <parent link="base_wheel_link" />
             <child link="${name}_wheel" />
             <origin
-                xyz="0 ${flag * base_link_radius} ${-(earth_space + base_link_length / 2 - wheel_radius) }" />
+                xyz="0 ${flag * base_wheel_link_radius} ${-(earth_space + base_wheel_link_length / 2 - wheel_radius) }" />
             <axis xyz="0 1 0" />
         </joint>
@@ -110,9 +110,9 @@
             <xacro:sphere_inertial_matrix m="${support_wheel_m}" r="${support_wheel_radius}" />
         </link>
-        <joint name="${name}_wheel2base_link" type="continuous">
-            <parent link="base_link" />
+        <joint name="${name}_wheel2base_wheel_link" type="continuous">
+            <parent link="base_wheel_link" />
             <child link="${name}_wheel" />
             <origin
-                xyz="${flag * (base_link_radius - support_wheel_radius)} 0 ${-(base_link_length / 2 + earth_space / 2)}" />
+                xyz="${flag * (base_wheel_link_radius - support_wheel_radius)} 0 ${-(base_wheel_link_length / 2 + earth_space / 2)}" />
             <axis xyz="1 1 1" />
         </joint>
@@ -124,10 +124,11 @@
     <xacro:add_support_wheel name="back" flag="-1" />
     <!-- 包含sunday机械臂 -->
-    <xacro:include filename="path/to/sunday.xacro" />
+    <xacro:include filename="$(find sunday_description)/urdf/sunday.xacro" />
     <!-- 设置base_link和sunday之间的连接 -->
     <joint name="base_to_sunday" type="fixed">
-        <parent link="base_link" /> <!-- base_wheel的基链接 -->
-        <child link="base_footprint" /> <!-- sunday的基链接 -->
-        <origin xyz="0 0 ${base_link_length / 2}" rpy="0 0 0" /> <!-- 根据需要调整位置和姿态 -->
+        <parent link="base_wheel_link" /> <!-- base_wheel的基链接 -->
+        <child link="world" /> <!-- sunday的基链接 -->
+        <!-- TODO: 调整wheel和sunday的相对位置 -->
+        <origin xyz="0 0 ${base_wheel_link_length / 2}" rpy="0 0 0" /> <!-- 根据需要调整位置和姿态 -->
     </joint>
 </robot>

File: src/my_robot_navigation/urdf/xacro/camera.xacro (robot description, xacro)
@@ -12,5 +12,5 @@
         name="camera_y" value="0.0" /> <!-- 摄像头安装的y坐标 -->
     <xacro:property name="camera_z"
-        value="${base_link_length / 2 + camera_height / 2}" /> <!--
+        value="${base_wheel_link_length / 2 + camera_height / 2}" /> <!--
     摄像头安装的z坐标:底盘高度 / 2 + 摄像头高度 / 2  -->
     <xacro:property name="camera_m"
@@ -34,6 +34,6 @@
             h="${camera_height}" />
     </link>
-    <joint name="camera2base_link" type="fixed">
-        <parent link="base_link" />
+    <joint name="camera2base_wheel_link" type="fixed">
+        <parent link="base_wheel_link" />
         <child link="camera" />
         <origin xyz="${camera_x} ${camera_y} ${camera_z}" />

File: src/my_robot_navigation/urdf/xacro/laser.xacro (robot description, xacro)
@@ -5,5 +5,5 @@
     <xacro:property name="support_x" value="0.0" /> <!-- 支架安装的x坐标 -->
     <xacro:property name="support_y" value="0.0" /> <!-- 支架安装的y坐标 -->
-    <xacro:property name="support_z" value="${base_link_length / 2 + support_length / 2}" /> <!--
+    <xacro:property name="support_z" value="${base_wheel_link_length / 2 + support_length / 2}" /> <!--
     支架安装的z坐标:底盘高度 / 2 + 支架高度 / 2  -->
     <xacro:property name="support_m" value="0.02" /> <!-- 支架质量 -->
@@ -26,6 +26,6 @@
         <xacro:cylinder_inertial_matrix m="${support_m}" r="${support_radius}" h="${support_length}" />
     </link>
-    <joint name="support2base_link" type="fixed">
-        <parent link="base_link" />
+    <joint name="support2base_wheel_link" type="fixed">
+        <parent link="base_wheel_link" />
         <child link="support" />
         <origin xyz="${support_x} ${support_y} ${support_z}" />

File: src/my_robot_navigation/urdf/xacro/move.xacro (robot description, xacro)
@@ -16,6 +16,6 @@
     </xacro:macro>
     <!-- 每一个驱动轮都需要配置传动装置 -->
-    <xacro:joint_trans joint_name="left_wheel2base_link" />
-    <xacro:joint_trans joint_name="right_wheel2base_link" />
+    <xacro:joint_trans joint_name="left_wheel2base_wheel_link" />
+    <xacro:joint_trans joint_name="right_wheel2base_wheel_link" />
     <!-- 控制器 -->
     <gazebo>
@@ -29,7 +29,7 @@
             <updateRate>100.0</updateRate>
             <legacyMode>true</legacyMode>
-            <leftJoint>left_wheel2base_link</leftJoint> <!-- 左轮 -->
-            <rightJoint>right_wheel2base_link</rightJoint> <!-- 右轮 -->
-            <wheelSeparation>${base_link_radius * 2}</wheelSeparation> <!-- 车轮间距 -->
+            <leftJoint>left_wheel2base_wheel_link</leftJoint> <!-- 左轮 -->
+            <rightJoint>right_wheel2base_wheel_link</rightJoint> <!-- 右轮 -->
+            <wheelSeparation>${base_wheel_link_radius * 2}</wheelSeparation> <!-- 车轮间距 -->
             <wheelDiameter>${wheel_radius * 2}</wheelDiameter> <!-- 车轮直径 -->
             <broadcastTF>1</broadcastTF>
@@ -39,5 +39,5 @@
             <odometryFrame>odom</odometryFrame>
             <odometryTopic>odom</odometryTopic> <!-- 里程计话题 -->
-            <robotBaseFrame>base_footprint</robotBaseFrame> <!-- 根坐标系 -->
+            <robotBaseFrame>base_wheel_footprint</robotBaseFrame> <!-- 根坐标系 -->
         </plugin>
     </gazebo>

Commit message: Refactor launch files and scripts for YOLOv5 integration

File: src/my_robot_navigation/urdf/xacro/base_wheel.xacro (robot description, xacro)
@@ -14,12 +14,4 @@
     <xacro:property name="earth_space" value="0.015" /> <!-- 离地间距 -->
     <xacro:property name="base_wheel_link_m" value="0.5" /> <!-- 质量  -->
-    <!-- 底盘 -->
-    <link name="base_wheel_footprint">
-        <visual>
-            <geometry>
-                <sphere radius="${base_wheel_footprint_radius}" />
-            </geometry>
-        </visual>
-    </link>
     <link name="base_wheel_link">
         <visual>
@@ -43,9 +35,4 @@
             h="${base_wheel_link_length}" />
     </link>
-    <joint name="base_wheel_link2base_wheel_footprint" type="fixed">
-        <parent link="base_wheel_footprint" />
-        <child link="base_wheel_link" />
-        <origin xyz="0 0 ${earth_space + base_wheel_link_length / 2 }" />
-    </joint>
     <gazebo reference="base_wheel_link">
         <!-- 与rviz不同（3）：重新设置颜色 -->
@@ -123,12 +110,3 @@
     <xacro:add_support_wheel name="front" flag="1" />
     <xacro:add_support_wheel name="back" flag="-1" />
-    <!-- 包含sunday机械臂 -->
-    <xacro:include filename="$(find sunday_description)/urdf/sunday.xacro" />
-    <!-- 设置base_link和sunday之间的连接 -->
-    <joint name="base_to_sunday" type="fixed">
-        <parent link="base_wheel_link" /> <!-- base_wheel的基链接 -->
-        <child link="world" /> <!-- sunday的基链接 -->
-        <!-- TODO: 调整wheel和sunday的相对位置 -->
-        <origin xyz="0 0 ${base_wheel_link_length / 2}" rpy="0 0 0" /> <!-- 根据需要调整位置和姿态 -->
-    </joint>
 </robot>

File: src/my_robot_navigation/urdf/xacro/move.xacro (robot description, xacro)
@@ -39,5 +39,5 @@
             <odometryFrame>odom</odometryFrame>
             <odometryTopic>odom</odometryTopic> <!-- 里程计话题 -->
-            <robotBaseFrame>base_wheel_footprint</robotBaseFrame> <!-- 根坐标系 -->
+            <robotBaseFrame>world</robotBaseFrame> <!-- 根坐标系 -->
         </plugin>
     </gazebo>

File: src/sunday/sunday_description/urdf/sunday.xacro (robot description, xacro)
@@ -402,4 +402,14 @@
       xyz="0 0 0" />
   </joint> -->
+  <!-- include robot.xacro -->
+  <xacro:include filename="$(find my_robot_navigation)/urdf/robot.xacro" />
+  <!-- joint -->
+  <joint name="world2base_wheel_link" type="fixed">
+    <origin
+      xyz="0 0 0"
+      rpy="0 0 0" />
+    <parent link="world" />
+    <child link="base_wheel_link" />
+  </joint>
   <!-- Used for fixing robot to Gazebo 'base_link' -->
   <link name="world" />
