Commit message: Refactor launch files and scripts for YOLOv5 integration

File: src/my_robot_navigation/urdf/robot.xacro (robot description, xacro)
@@ -3,5 +3,5 @@
   <xacro:include filename="xacro/inertial.xacro" />
   <xacro:include filename="xacro/base_wheel.xacro" />
-  <xacro:include filename="xacro/camera.xacro" />
+  <!-- <xacro:include filename="xacro/camera.xacro" /> -->
   <xacro:include filename="xacro/laser.xacro" />
   <xacro:include filename="xacro/move.xacro" />

File: src/my_robot_navigation/urdf/xacro/base_wheel.xacro (robot description, xacro)
@@ -10,8 +10,8 @@
     <!-- 底盘属性 -->
     <xacro:property name="base_wheel_footprint_radius" value="0.001" /> <!-- base_wheel_footprint 半径  -->
-    <xacro:property name="base_wheel_link_radius" value="0.1" /> <!-- base_wheel_link 半径 -->
-    <xacro:property name="base_wheel_link_length" value="0.08" /> <!-- base_wheel_link 长 -->
-    <xacro:property name="earth_space" value="0.015" /> <!-- 离地间距 -->
-    <xacro:property name="base_wheel_link_m" value="0.5" /> <!-- 质量  -->
+    <xacro:property name="base_wheel_link_radius" value="0.3" /> <!-- base_wheel_link 半径 -->
+    <xacro:property name="base_wheel_link_length" value="0.3" /> <!-- base_wheel_link 长 -->
+    <xacro:property name="earth_space" value="0.15" /> <!-- 离地间距 -->
+    <xacro:property name="base_wheel_link_m" value="1.0" /> <!-- 质量  -->
     <!-- 底盘 -->
     <link name="base_wheel_footprint">
@@ -54,7 +54,7 @@
     <!-- 驱动轮 -->
     <!-- 驱动轮属性 -->
-    <xacro:property name="wheel_radius" value="0.0325" /> <!-- 半径 -->
-    <xacro:property name="wheel_length" value="0.015" /> <!-- 宽度 -->
-    <xacro:property name="wheel_m" value="0.05" /> <!-- 质量  -->
+    <xacro:property name="wheel_radius" value="0.1" /> <!-- 半径 -->
+    <xacro:property name="wheel_length" value="0.045" /> <!-- 宽度 -->
+    <xacro:property name="wheel_m" value="0.10" /> <!-- 质量  -->
     <!-- 驱动轮宏实现 -->
     <xacro:macro name="add_wheels" params="name flag">
@@ -123,12 +123,3 @@
     <xacro:add_support_wheel name="front" flag="1" />
     <xacro:add_support_wheel name="back" flag="-1" />
-    <!-- 包含sunday机械臂 -->
-    <xacro:include filename="$(find sunday_description)/urdf/sunday.xacro" />
-    <!-- 设置base_link和sunday之间的连接 -->
-    <joint name="base_to_sunday" type="fixed">
-        <parent link="base_wheel_link" /> <!-- base_wheel的基链接 -->
-        <child link="world" /> <!-- sunday的基链接 -->
-        <!-- TODO: 调整wheel和sunday的相对位置 -->
-        <origin xyz="0 0 ${base_wheel_link_length / 2}" rpy="0 0 0" /> <!-- 根据需要调整位置和姿态 -->
-    </joint>
 </robot>

File: src/sunday/sunday_description/urdf/sunday.xacro (robot description, xacro)
@@ -7,4 +7,12 @@
   <link name="base_footprint">
   </link>
+  <!-- include robot.xacro -->
+  <xacro:include filename="$(find my_robot_navigation)/urdf/robot.xacro" />
+  <!-- joint -->
+  <joint name="world2base_wheel_footprint" type="fixed">
+    <origin xyz="0 0 0" rpy="0 0 0" />
+    <parent link="base_footprint" />
+    <child link="base_wheel_footprint" />
+  </joint>
   <link name="base_link">
     <inertial>
@@ -42,5 +50,7 @@
     <parent link="base_footprint" />
     <child link="base_link" />
-    <origin xyz="0 0 0.032" rpy="0 0 0" />
+    <origin
+      xyz="${base_wheel_link_radius} ${base_wheel_link_radius / 2} ${base_wheel_link_length + earth_space + 0.032}"
+      rpy="0 0 0" />
   </joint>
   <link name="link_1">
@@ -406,5 +416,5 @@
   <joint name="fixed" type="fixed">
     <origin
-      xyz="0 0 1.1"
+      xyz="0 1.1 0"
       rpy="0 0 0" />
     <parent link="world" />

Commit message: Refactor launch files and scripts for YOLOv5 integration

File: src/my_robot_navigation/urdf/robot.xacro (robot description, xacro)
@@ -3,6 +3,15 @@
   <xacro:include filename="xacro/inertial.xacro" />
   <xacro:include filename="xacro/base_wheel.xacro" />
-  <xacro:include filename="xacro/camera.xacro" />
+  <!-- <xacro:include filename="xacro/camera.xacro" /> -->
   <xacro:include filename="xacro/laser.xacro" />
   <xacro:include filename="xacro/move.xacro" />
+  <!-- sunday.xacro -->
+  <xacro:include filename="$(find sunday_description)/urdf/sunday.xacro" />
+  <joint name="sunday2base_car_link" type="fixed">
+    <parent link="base_car_link" />
+    <child link="base_footprint" />
+    <origin
+      xyz="${base_car_link_radius / 3} ${base_car_link_radius / 2} 0"
+      rpy="0 0 0" />
+  </joint>
 </robot>

File: src/my_robot_navigation/urdf/xacro/base_wheel.xacro (robot description, xacro)
@@ -9,21 +9,23 @@
     </material>
     <!-- 底盘属性 -->
-    <xacro:property name="base_footprint_radius" value="0.001" /> <!-- base_footprint 半径  -->
-    <xacro:property name="base_link_radius" value="0.1" /> <!-- base_link 半径 -->
-    <xacro:property name="base_link_length" value="0.08" /> <!-- base_link 长 -->
-    <xacro:property name="earth_space" value="0.015" /> <!-- 离地间距 -->
-    <xacro:property name="base_link_m" value="0.5" /> <!-- 质量  -->
+    <xacro:property name="scale" value="3" />
+    <xacro:property name="base_car_footprint_radius" value="${scale * 0.001}" /> <!--
+    base_car_footprint 半径  -->
+    <xacro:property name="base_car_link_radius" value="${scale * 0.1}" /> <!-- base_car_link 半径 -->
+    <xacro:property name="base_car_link_length" value="${scale * 0.08}" /> <!-- base_car_link 长 -->
+    <xacro:property name="earth_space" value="${scale * 0.015}" /> <!-- 离地间距 -->
+    <xacro:property name="base_car_link_m" value="${scale * 1}" /> <!-- 质量  -->
     <!-- 底盘 -->
-    <link name="base_footprint">
+    <link name="base_car_footprint">
         <visual>
             <geometry>
-                <sphere radius="${base_footprint_radius}" />
+                <sphere radius="${base_car_footprint_radius}" />
             </geometry>
         </visual>
     </link>
-    <link name="base_link">
+    <link name="base_car_link">
         <visual>
             <geometry>
-                <cylinder radius="${base_link_radius}" length="${base_link_length}" />
+                <cylinder radius="${base_car_link_radius}" length="${base_car_link_length}" />
             </geometry>
             <origin xyz="0 0 0" rpy="0 0 0" />
@@ -35,18 +37,18 @@
         <collision>
             <geometry>
-                <cylinder radius="${base_link_radius}" length="${base_link_length}" />
+                <cylinder radius="${base_car_link_radius}" length="${base_car_link_length}" />
             </geometry>
             <origin xyz="0 0 0" rpy="0 0 0" />
         </collision>
         <!-- 与rviz不同（2）：使用在head.xacro中封装过的inertial标签 -->
-        <xacro:cylinder_inertial_matrix m="${base_link_m}" r="${base_link_radius}"
-            h="${base_link_length}" />
+        <xacro:cylinder_inertial_matrix m="${base_car_link_m}" r="${base_car_link_radius}"
+            h="${base_car_link_length}" />
     </link>
-    <joint name="base_link2base_footprint" type="fixed">
-        <parent link="base_footprint" />
-        <child link="base_link" />
-        <origin xyz="0 0 ${earth_space + base_link_length / 2 }" />
+    <joint name="base_car_link2base_car_footprint" type="fixed">
+        <parent link="base_car_footprint" />
+        <child link="base_car_link" />
+        <origin xyz="0 0 ${earth_space + base_car_link_length / 2 }" />
     </joint>
-    <gazebo reference="base_link">
+    <gazebo reference="base_car_link">
         <!-- 与rviz不同（3）：重新设置颜色 -->
         <material>Gazebo/Yellow</material>
@@ -54,7 +56,7 @@
     <!-- 驱动轮 -->
     <!-- 驱动轮属性 -->
-    <xacro:property name="wheel_radius" value="0.0325" /> <!-- 半径 -->
-    <xacro:property name="wheel_length" value="0.015" /> <!-- 宽度 -->
-    <xacro:property name="wheel_m" value="0.05" /> <!-- 质量  -->
+    <xacro:property name="wheel_radius" value="${scale * 0.0325}" /> <!-- 半径 -->
+    <xacro:property name="wheel_length" value="${scale * 0.015}" /> <!-- 宽度 -->
+    <xacro:property name="wheel_m" value="${scale * 0.05}" /> <!-- 质量  -->
     <!-- 驱动轮宏实现 -->
     <xacro:macro name="add_wheels" params="name flag">
@@ -75,9 +77,9 @@
             <xacro:cylinder_inertial_matrix m="${wheel_m}" r="${wheel_radius}" h="${wheel_length}" />
         </link>
-        <joint name="${name}_wheel2base_link" type="continuous">
-            <parent link="base_link" />
+        <joint name="${name}_wheel2base_car_link" type="continuous">
+            <parent link="base_car_link" />
             <child link="${name}_wheel" />
             <origin
-                xyz="0 ${flag * base_link_radius} ${-(earth_space + base_link_length / 2 - wheel_radius) }" />
+                xyz="0 ${flag * base_car_link_radius} ${-(earth_space + base_car_link_length / 2 - wheel_radius) }" />
             <axis xyz="0 1 0" />
         </joint>
@@ -90,6 +92,6 @@
     <!-- 支撑轮 -->
     <!-- 支撑轮属性 -->
-    <xacro:property name="support_wheel_radius" value="0.0075" /> <!-- 支撑轮半径 -->
-    <xacro:property name="support_wheel_m" value="0.03" /> <!-- 质量  -->
+    <xacro:property name="support_wheel_radius" value="${scale * 0.0075}" /> <!-- 支撑轮半径 -->
+    <xacro:property name="support_wheel_m" value="0.1" /> <!-- 质量  -->
     <!-- 支撑轮宏 -->
     <xacro:macro name="add_support_wheel" params="name flag">
@@ -110,9 +112,9 @@
             <xacro:sphere_inertial_matrix m="${support_wheel_m}" r="${support_wheel_radius}" />
         </link>
-        <joint name="${name}_wheel2base_link" type="continuous">
-            <parent link="base_link" />
+        <joint name="${name}_wheel2base_car_link" type="continuous">
+            <parent link="base_car_link" />
             <child link="${name}_wheel" />
             <origin
-                xyz="${flag * (base_link_radius - support_wheel_radius)} 0 ${-(base_link_length / 2 + earth_space / 2)}" />
+                xyz="${flag * (base_car_link_radius - support_wheel_radius)} 0 ${-(base_car_link_length / 2 + earth_space / 2)}" />
             <axis xyz="1 1 1" />
         </joint>

File: src/my_robot_navigation/urdf/xacro/laser.xacro (robot description, xacro)
@@ -1,11 +1,13 @@
 <robot name="my_laser" xmlns:xacro="http://wiki.ros.org/xacro">
     <!-- 雷达支架 -->
-    <xacro:property name="support_length" value="0.15" /> <!-- 支架长度 -->
-    <xacro:property name="support_radius" value="0.01" /> <!-- 支架半径 -->
+    <!-- [ ]: 尺度 -->
+    <xacro:property name="scale" value="2" />
+    <xacro:property name="support_length" value="${scale * 0.15}" /> <!-- 支架长度 -->
+    <xacro:property name="support_radius" value="${scale * 0.01}" /> <!-- 支架半径 -->
     <xacro:property name="support_x" value="0.0" /> <!-- 支架安装的x坐标 -->
     <xacro:property name="support_y" value="0.0" /> <!-- 支架安装的y坐标 -->
-    <xacro:property name="support_z" value="${base_link_length / 2 + support_length / 2}" /> <!--
+    <xacro:property name="support_z" value="${base_car_link_length / 2 + support_length / 2}" /> <!--
     支架安装的z坐标:底盘高度 / 2 + 支架高度 / 2  -->
-    <xacro:property name="support_m" value="0.02" /> <!-- 支架质量 -->
+    <xacro:property name="support_m" value="${scale * 0.02}" /> <!-- 支架质量 -->
     <link name="support">
         <visual>
@@ -26,6 +28,6 @@
         <xacro:cylinder_inertial_matrix m="${support_m}" r="${support_radius}" h="${support_length}" />
     </link>
-    <joint name="support2base_link" type="fixed">
-        <parent link="base_link" />
+    <joint name="support2base_car_link" type="fixed">
+        <parent link="base_car_link" />
         <child link="support" />
         <origin xyz="${support_x} ${support_y} ${support_z}" />

File: src/my_robot_navigation/urdf/xacro/move.xacro (robot description, xacro)
@@ -16,6 +16,6 @@
     </xacro:macro>
     <!-- 每一个驱动轮都需要配置传动装置 -->
-    <xacro:joint_trans joint_name="left_wheel2base_link" />
-    <xacro:joint_trans joint_name="right_wheel2base_link" />
+    <xacro:joint_trans joint_name="left_wheel2base_car_link" />
+    <xacro:joint_trans joint_name="right_wheel2base_car_link" />
     <!-- 控制器 -->
     <gazebo>
@@ -29,15 +29,15 @@
             <updateRate>100.0</updateRate>
             <legacyMode>true</legacyMode>
-            <leftJoint>left_wheel2base_link</leftJoint> <!-- 左轮 -->
-            <rightJoint>right_wheel2base_link</rightJoint> <!-- 右轮 -->
-            <wheelSeparation>${base_link_radius * 2}</wheelSeparation> <!-- 车轮间距 -->
+            <leftJoint>left_wheel2base_car_link</leftJoint> <!-- 左轮 -->
+            <rightJoint>right_wheel2base_car_link</rightJoint> <!-- 右轮 -->
+            <wheelSeparation>${base_car_link_radius * 2}</wheelSeparation> <!-- 车轮间距 -->
             <wheelDiameter>${wheel_radius * 2}</wheelDiameter> <!-- 车轮直径 -->
             <broadcastTF>1</broadcastTF>
-            <wheelTorque>30</wheelTorque>
-            <wheelAcceleration>1.8</wheelAcceleration>
+            <wheelTorque>300</wheelTorque>
+            <wheelAcceleration>10.8</wheelAcceleration>
             <commandTopic>cmd_vel</commandTopic> <!-- 运动控制话题 -->
             <odometryFrame>odom</odometryFrame>
             <odometryTopic>odom</odometryTopic> <!-- 里程计话题 -->
-            <robotBaseFrame>base_footprint</robotBaseFrame> <!-- 根坐标系 -->
+            <robotBaseFrame>base_car_footprint</robotBaseFrame> <!-- 根坐标系 -->
         </plugin>
     </gazebo>

File: src/sunday/sunday_description/urdf/sunday.xacro (robot description, xacro)
@@ -403,12 +403,12 @@
   </joint> -->
   <!-- Used for fixing robot to Gazebo 'base_link' -->
-  <link name="world" />
+  <!-- <link name="world" />
   <joint name="fixed" type="fixed">
     <origin
-      xyz="0 0 1.1"
+      xyz="0 0 0"
       rpy="0 0 0" />
     <parent link="world" />
     <child link="base_footprint" />
-  </joint>
+  </joint> -->
   <!-- <xacro:include filename="$(find sunday_description)/urdf/realsense/realsense.xacro"/> -->
   <xacro:include filename="$(find realsense_ros_gazebo)/xacro/depthcam.xacro" />

Commit message: Refactor robot.xacro and laser.xacro for YOLOv5 integration

File: src/my_robot_navigation/urdf/robot.xacro (robot description, xacro)
@@ -12,5 +12,5 @@
     <child link="base_footprint" />
     <origin
-      xyz="${base_car_link_radius / 3} ${base_car_link_radius / 2} 0"
+      xyz="${base_car_link_radius / 3} ${base_car_link_radius / 2} -0.032"
       rpy="0 0 0" />
   </joint>

File: src/my_robot_navigation/urdf/xacro/arm.xacro (robot description, xacro)
@@ -1,4 +1,4 @@
 <?xml version="1.0"?>
-<robot name="simple_arm" xmlns:xacro="http://ros.org/wiki/xacro">
+<robot name="my_robot_arm" xmlns:xacro="http://www.ros.org/wiki/xacro">
     <!-- Define some constants -->
     <xacro:property name="arm_length" value="1.0" />
@@ -6,6 +6,4 @@
     <xacro:property name="gripper_length" value="0.2" />
     <xacro:property name="gripper_radius" value="0.02" />
-    <xacro:property name="finger_length" value="0.1" />
-    <xacro:property name="finger_radius" value="0.01" />
     <!-- Base link -->
     <link name="base_link">
@@ -14,80 +12,72 @@
                 <cylinder length="0.1" radius="0.1" />
             </geometry>
-            <material name="grey">
-                <color rgba="0.5 0.5 0.5 1.0" />
-            </material>
+            <material name="blue" />
         </visual>
     </link>
-    <!-- Arm link -->
-    <link name="arm_link">
+    <!-- Joint 1 -->
+    <joint name="joint1" type="revolute">
+        <parent link="base_link" />
+        <child link="link1" />
+        <origin xyz="0 0 0.05" rpy="0 0 0" />
+        <axis xyz="0 0 1" />
+        <limit lower="-1.57" upper="1.57" effort="10" velocity="1" />
+    </joint>
+    <!-- Link 1 -->
+    <link name="link1">
         <visual>
             <geometry>
                 <cylinder length="${arm_length}" radius="${arm_radius}" />
             </geometry>
-            <material name="blue">
-                <color rgba="0.0 0.0 1.0 1.0" />
-            </material>
+            <material name="green" />
         </visual>
     </link>
-    <!-- Gripper link -->
-    <link name="gripper_link">
+    <!-- Joint 2 -->
+    <joint name="joint2" type="revolute">
+        <parent link="link1" />
+        <child link="link2" />
+        <origin xyz="0 0 ${arm_length}" rpy="0 0 0" />
+        <axis xyz="0 1 0" />
+        <limit lower="-1.57" upper="1.57" effort="10" velocity="1" />
+    </joint>
+    <!-- Link 2 -->
+    <link name="link2">
+        <visual>
+            <geometry>
+                <cylinder length="${arm_length}" radius="${arm_radius}" />
+            </geometry>
+            <material name="red" />
+        </visual>
+    </link>
+    <!-- Joint 3 -->
+    <joint name="joint3" type="revolute">
+        <parent link="link2" />
+        <child link="link3" />
+        <origin xyz="0 0 ${arm_length}" rpy="0 0 0" />
+        <axis xyz="0 1 0" />
+        <limit lower="-1.57" upper="1.57" effort="10" velocity="1" />
+    </joint>
+    <!-- Link 3 -->
+    <link name="link3">
+        <visual>
+            <geometry>
+                <cylinder length="${arm_length}" radius="${arm_radius}" />
+            </geometry>
+            <material name="yellow" />
+        </visual>
+    </link>
+    <!-- Gripper Joint -->
+    <joint name="gripper_joint" type="fixed">
+        <parent link="link3" />
+        <child link="gripper" />
+        <origin xyz="0 0 ${arm_length}" rpy="0 0 0" />
+    </joint>
+    <!-- Gripper -->
+    <link name="gripper">
         <visual>
             <geometry>
                 <cylinder length="${gripper_length}" radius="${gripper_radius}" />
             </geometry>
-            <material name="red">
-                <color rgba="1.0 0.0 0.0 1.0" />
-            </material>
+            <material name="gray" />
         </visual>
     </link>
-    <!-- Finger links -->
-    <link name="left_finger">
-        <visual>
-            <geometry>
-                <cylinder length="${finger_length}" radius="${finger_radius}" />
-            </geometry>
-            <material name="green">
-                <color rgba="0.0 1.0 0.0 1.0" />
-            </material>
-        </visual>
-    </link>
-    <link name="right_finger">
-        <visual>
-            <geometry>
-                <cylinder length="${finger_length}" radius="${finger_radius}" />
-            </geometry>
-            <material name="green">
-                <color rgba="0.0 1.0 0.0 1.0" />
-            </material>
-        </visual>
-    </link>
-    <!-- Joints -->
-    <joint name="base_to_arm" type="revolute">
-        <parent link="base_link" />
-        <child link="arm_link" />
-        <origin xyz="0 0 0.05" rpy="0 0 0" />
-        <axis xyz="0 1 0" />
-        <limit lower="-1.57" upper="1.57" effort="10" velocity="1.0" />
-    </joint>
-    <joint name="arm_to_gripper" type="revolute">
-        <parent link="arm_link" />
-        <child link="gripper_link" />
-        <origin xyz="0 0 ${arm_length/2}" rpy="0 0 0" />
-        <axis xyz="0 1 0" />
-        <limit lower="-1.57" upper="1.57" effort="10" velocity="1.0" />
-    </joint>
-    <joint name="gripper_to_left_finger" type="prismatic">
-        <parent link="gripper_link" />
-        <child link="left_finger" />
-        <origin xyz="0 ${gripper_radius} ${gripper_length/2}" rpy="0 0 0" />
-        <axis xyz="0 1 0" />
-        <limit lower="0" upper="${gripper_radius}" effort="10" velocity="1.0" />
-    </joint>
-    <joint name="gripper_to_right_finger" type="prismatic">
-        <parent link="gripper_link" />
-        <child link="right_finger" />
-        <origin xyz="0 -${gripper_radius} ${gripper_length/2}" rpy="0 0 0" />
-        <axis xyz="0 -1 0" />
-        <limit lower="0" upper="${gripper_radius}" effort="10" velocity="1.0" />
-    </joint>
 </robot>

File: src/my_robot_navigation/urdf/xacro/base_wheel.xacro (robot description, xacro)
@@ -15,5 +15,5 @@
     <xacro:property name="base_car_link_length" value="${scale * 0.08}" /> <!-- base_car_link 长 -->
     <xacro:property name="earth_space" value="${scale * 0.015}" /> <!-- 离地间距 -->
-    <xacro:property name="base_car_link_m" value="${scale * 1}" /> <!-- 质量  -->
+    <xacro:property name="base_car_link_m" value="${scale * 0.8}" /> <!-- 质量  -->
     <!-- 底盘 -->
     <link name="base_car_footprint">

File: src/my_robot_navigation/urdf/xacro/laser.xacro (robot description, xacro)
@@ -2,5 +2,5 @@
     <!-- 雷达支架 -->
     <!-- [ ]: 尺度 -->
-    <xacro:property name="scale" value="2" />
+    <xacro:property name="scale" value="3" />
     <xacro:property name="support_length" value="${scale * 0.15}" /> <!-- 支架长度 -->
     <xacro:property name="support_radius" value="${scale * 0.01}" /> <!-- 支架半径 -->

File: src/my_robot_navigation/urdf/xacro/move.xacro (robot description, xacro)
@@ -22,6 +22,6 @@
         <plugin name="differential_drive_controller" filename="libgazebo_ros_diff_drive.so">
             <rosDebugLevel>Debug</rosDebugLevel>
-            <publishWheelTF>true</publishWheelTF>
-            <robotNamespace>/</robotNamespace>
+            <publishWheelTF>false</publishWheelTF>
+            <robotNamespace>/car</robotNamespace>
             <publishTf>1</publishTf>
             <publishWheelJointState>true</publishWheelJointState>
