Commit message: nav and graps success ! ! !

File: src/my_robot_navigation/urdf/robot.xacro (robot description, xacro)
@@ -12,5 +12,5 @@
     <child link="base_footprint" />
     <origin
-      xyz="${base_car_link_radius / 3} ${base_car_link_radius / 2} -0.032"
+      xyz="${base_car_link_radius / 3} ${base_car_link_radius / 2} 0.2"
       rpy="0 0 0" />
   </joint>

File: src/my_robot_navigation/urdf/xacro/base_wheel.xacro (robot description, xacro)
@@ -15,5 +15,5 @@
     <xacro:property name="base_car_link_length" value="${scale * 0.08}" /> <!-- base_car_link 长 -->
     <xacro:property name="earth_space" value="${scale * 0.015}" /> <!-- 离地间距 -->
-    <xacro:property name="base_car_link_m" value="${scale * 0.8}" /> <!-- 质量  -->
+    <xacro:property name="base_car_link_m" value="${scale * 0.5}" /> <!-- 质量  -->
     <!-- 底盘 -->
     <link name="base_car_footprint">
@@ -93,5 +93,5 @@
     <!-- 支撑轮属性 -->
     <xacro:property name="support_wheel_radius" value="${scale * 0.0075}" /> <!-- 支撑轮半径 -->
-    <xacro:property name="support_wheel_m" value="0.1" /> <!-- 质量  -->
+    <xacro:property name="support_wheel_m" value="0.03" /> <!-- 质量  -->
     <!-- 支撑轮宏 -->
     <xacro:macro name="add_support_wheel" params="name flag">

File: src/my_robot_navigation/urdf/xacro/move.xacro (robot description, xacro)
@@ -20,24 +20,10 @@
     <!-- 控制器 -->
     <gazebo>
-        <plugin name="differential_drive_controller" filename="libgazebo_ros_diff_drive.so">
-            <rosDebugLevel>Debug</rosDebugLevel>
-            <publishWheelTF>false</publishWheelTF>
-            <robotNamespace>/car</robotNamespace>
-            <publishTf>1</publishTf>
-            <publishWheelJointState>true</publishWheelJointState>
-            <alwaysOn>true</alwaysOn>
-            <updateRate>100.0</updateRate>
-            <legacyMode>true</legacyMode>
-            <leftJoint>left_wheel2base_car_link</leftJoint> <!-- 左轮 -->
-            <rightJoint>right_wheel2base_car_link</rightJoint> <!-- 右轮 -->
-            <wheelSeparation>${base_car_link_radius * 2}</wheelSeparation> <!-- 车轮间距 -->
-            <wheelDiameter>${wheel_radius * 2}</wheelDiameter> <!-- 车轮直径 -->
-            <broadcastTF>1</broadcastTF>
-            <wheelTorque>300</wheelTorque>
-            <wheelAcceleration>10.8</wheelAcceleration>
-            <commandTopic>cmd_vel</commandTopic> <!-- 运动控制话题 -->
+        <plugin name="object_controller" filename="libgazebo_ros_planar_move.so">
+            <commandTopic>cmd_vel</commandTopic>
+            <odometryTopic>odom</odometryTopic>
             <odometryFrame>odom</odometryFrame>
-            <odometryTopic>odom</odometryTopic> <!-- 里程计话题 -->
-            <robotBaseFrame>base_car_footprint</robotBaseFrame> <!-- 根坐标系 -->
+            <odometryRate>20.0</odometryRate>
+            <robotBaseFrame>base_footprint</robotBaseFrame>
         </plugin>
     </gazebo>

Commit message: Refactor robot.xacro and laser.xacro for YOLOv5 integration

File: src/my_robot_navigation/urdf/robot.xacro (robot description, xacro)
@@ -12,5 +12,5 @@
     <child link="base_footprint" />
     <origin
-      xyz="${base_car_link_radius / 3} ${base_car_link_radius / 2} 0.2"
+      xyz="${base_car_link_radius / 3} ${base_car_link_radius / 2} ${earth_space + base_car_link_length}"
       rpy="0 0 0" />
   </joint>

File: src/my_robot_navigation/urdf/xacro/base_wheel.xacro (robot description, xacro)
@@ -13,7 +13,7 @@
     base_car_footprint 半径  -->
     <xacro:property name="base_car_link_radius" value="${scale * 0.1}" /> <!-- base_car_link 半径 -->
-    <xacro:property name="base_car_link_length" value="${scale * 0.08}" /> <!-- base_car_link 长 -->
+    <xacro:property name="base_car_link_length" value="${scale * 0.03}" /> <!-- base_car_link 长 -->
     <xacro:property name="earth_space" value="${scale * 0.015}" /> <!-- 离地间距 -->
-    <xacro:property name="base_car_link_m" value="${scale * 0.5}" /> <!-- 质量  -->
+    <xacro:property name="base_car_link_m" value="${scale *1}" /> <!-- 质量  -->
     <!-- 底盘 -->
     <link name="base_car_footprint">

File: src/sunday/sunday_description/urdf/sunday.xacro (robot description, xacro)
@@ -12,5 +12,5 @@
         xyz="-0.0041595 -0.019776 0.12"
         rpy="0 0 0" />
-      <mass value="0.524001417146026" />
+      <mass value="0.0524001417146026" />
       <inertia ixx="1" ixy="0" ixz="0" iyy="1" iyz="0" izz="1" />
     </inertial>
@@ -42,5 +42,5 @@
     <parent link="base_footprint" />
     <child link="base_link" />
-    <origin xyz="0 0 0.032" rpy="0 0 0" />
+    <origin xyz="0 0 0" rpy="0 0 0" />
   </joint>
   <link name="link_1">
@@ -49,5 +49,5 @@
         xyz="4.4076E-07 0.0088489 0.03981"
         rpy="0 0 0" />
-      <mass value="0.166259789544396" />
+      <mass value="0.0166259789544396" />
       <inertia ixx="1" ixy="0" ixz="0" iyy="1" iyz="0" izz="1" />
     </inertial>
@@ -100,5 +100,5 @@
         xyz="5.2117E-07 0.050183 0.046384"
         rpy="0 0 0" />
-      <mass value="0.316094041078938" />
+      <mass value="0.0316094041078938" />
       <inertia ixx="1" ixy="0" ixz="0" iyy="1" iyz="0" izz="1" />
     </inertial>
@@ -151,5 +151,5 @@
         xyz="-2.3744E-06 0.013658 -0.095655"
         rpy="0 0 0" />
-      <mass value="0.323135746651779" />
+      <mass value="0.0323135746651779" />
       <inertia ixx="1" ixy="0" ixz="0" iyy="1" iyz="0" izz="1" />
     </inertial>
@@ -202,5 +202,5 @@
         xyz="-6.4344E-06 -0.026419 -0.014391"
         rpy="0 0 0" />
-      <mass value="0.174947986817189" />
+      <mass value="0.0174947986817189" />
       <inertia ixx="1" ixy="0" ixz="0" iyy="1" iyz="0" izz="1" />
     </inertial>
@@ -253,5 +253,5 @@
         xyz="0.00020466 -0.017155 -0.036587"
         rpy="0 0 0" />
-      <mass value="0.174947985033356" />
+      <mass value="0.0174947985033356" />
       <inertia ixx="1" ixy="0" ixz="0" iyy="1" iyz="0" izz="1" />
     </inertial>
